File: cinch_pinout.kicad_pcb (KiCad board)
At the start: 2 copper layers, 14.7 x 17.6 mm, 4 parts, among them J1 Conn, J2 Pinout

Commit message: Updated template for KiCAD 7
Parts:
- J1: footprint footprints:MJ2509N -> Chof747 Footprints:MJ2509N
